Commit message: working gazebo controllers

File: spot_arm_description/urdf/spot_arm.xacro (robot description, xacro)
@@ -4,4 +4,10 @@
 <xacro:include filename="$(find spot_arm_description)/urdf/spot_arm.trans" />
 <xacro:include filename="$(find spot_arm_description)/urdf/spot_arm.gazebo" />
+<!-- test -->
+<link name="world"/>
+<joint name="fixed_joint" type="fixed">
+    <parent link="world"/>
+    <child link="base_link"/>
+</joint>
 <link name="base_link">
   <inertial>

Commit message: Adapt arm urdf to match ros driver

File: spot_arm_description/urdf/spot_arm.xacro (robot description, xacro)
@@ -4,11 +4,59 @@
 <xacro:include filename="$(find spot_arm_description)/urdf/spot_arm.trans" />
 <xacro:include filename="$(find spot_arm_description)/urdf/spot_arm.gazebo" />
-<!-- test -->
 <link name="world"/>
-<joint name="fixed_joint" type="fixed">
+<joint name="base_arm_joint" type="fixed">
     <parent link="world"/>
-    <child link="base_link"/>
-</joint>
-<link name="base_link">
+    <child link="base_arm_link"/>
+</joint>
+<joint name="arm_joint1" type="revolute">
+  <origin rpy="0 0 0" xyz="0.0 0.0 0.065"/>
+  <parent link="base_arm_link"/>
+  <child link="link1"/>
+  <axis xyz="0.0 0.0 1.0"/>
+  <limit effort="100" lower="-3.141593" upper="2.617994" velocity="100"/>
+</joint>
+<joint name="arm_joint2" type="revolute">
+  <origin rpy="0 0 0" xyz="0.015 0.0 0.05"/>
+  <parent link="link1"/>
+  <child link="link2"/>
+  <axis xyz="-1.0 0.0 0.0"/>
+  <limit effort="100" lower="-3.665191" upper="0.0" velocity="100"/>
+</joint>
+<joint name="arm_joint3" type="revolute">
+  <origin rpy="0 0 0" xyz="0.002 0.3125 0.0"/>
+  <parent link="link2"/>
+  <child link="link3"/>
+  <axis xyz="1.0 0.0 0.0"/>
+  <limit effort="100" lower="0.0" upper="2.96706" velocity="100"/>
+</joint>
+<joint name="arm_joint4" type="revolute">
+  <origin rpy="0 0 0" xyz="-0.018 0.138 -0.0675"/>
+  <parent link="link3"/>
+  <child link="link4"/>
+  <axis xyz="0.0 1.0 0.0"/>
+  <limit effort="100" lower="-2.879793" upper="2.879793" velocity="100"/>
+</joint>
+<joint name="arm_joint5" type="revolute">
+  <origin rpy="0 0 0" xyz="-0.0475 0.24809 0.0"/>
+  <parent link="link4"/>
+  <child link="wrist"/>
+  <axis xyz="1.0 0.0 0.0"/>
+  <limit effort="100" lower="-1.570796" upper="1.570796" velocity="100"/>
+</joint>
+<joint name="arm_joint6" type="revolute">
+  <origin rpy="0 0 0" xyz="0.04 0.081 0.0"/>
+  <parent link="wrist"/>
+  <child link="gripper"/>
+  <axis xyz="-0.0 1.0 0.0"/>
+  <limit effort="100" lower="-2.96706" upper="2.96706" velocity="100"/>
+</joint>
+<joint name="arm_gripper" type="revolute">
+  <origin rpy="0 0 0" xyz="-0.86859 0.043915 -0.029"/>
+  <parent link="gripper"/>
+  <child link="finger"/>
+  <axis xyz="1.0 -0.0 0.0"/>
+  <limit effort="100" lower="-1.396263" upper="0.349066" velocity="100"/>
+</joint>
+<link name="base_arm_link">
   <inertial>
     <origin rpy="0 0 0" xyz="1.2371844231029972e-17 0.0 0.0325"/>
@@ -30,5 +78,65 @@
   </collision>
 </link>
-<link name="Part3_1">
+<link name="link1">
+  <inertial>
+    <origin rpy="0 0 0" xyz="0.05071972800114364 -1.0308563411658574e-17 0.04676911608650795"/>
+    <mass value="6.925827706354272"/>
+    <inertia ixx="0.01241" ixy="-0.0" ixz="-0.001047" iyy="0.010387" iyz="0.0" izz="0.012306"/>
+  </inertial>
+  <visual>
+    <origin rpy="0 0 0" xyz="-0.0 -0.0 -0.065"/>
+    <geometry>
+      <mesh filename="package://spot_arm_description/meshes/Part0_1.stl" scale="0.001 0.001 0.001"/>
+    </geometry>
+    <material name="silver"/>
+  </visual>
+  <collision>
+    <origin rpy="0 0 0" xyz="-0.0 -0.0 -0.065"/>
+    <geometry>
+      <mesh filename="package://spot_arm_description/meshes/Part0_1.stl" scale="0.001 0.001 0.001"/>
+    </geometry>
+  </collision>
+</link>
+<link name="link2">
+  <inertial>
+    <origin rpy="0 0 0" xyz="-0.0163095589512068 0.17540914221218962 0.0"/>
+    <mass value="12.658281999999998"/>
+    <inertia ixx="0.12979" ixy="0.002625" ixz="0.0" iyy="0.01004" iyz="0.0" izz="0.129493"/>
+  </inertial>
+  <visual>
+    <origin rpy="0 0 0" xyz="-0.015 -0.0 -0.115"/>
+    <geometry>
+      <mesh filename="package://spot_arm_description/meshes/Part1_1.stl" scale="0.001 0.001 0.001"/>
+    </geometry>
+    <material name="silver"/>
+  </visual>
+  <collision>
+    <origin rpy="0 0 0" xyz="-0.015 -0.0 -0.115"/>
+    <geometry>
+      <mesh filename="package://spot_arm_description/meshes/Part1_1.stl" scale="0.001 0.001 0.001"/>
+    </geometry>
+  </collision>
+</link>
+<link name="link3">
+  <inertial>
+    <origin rpy="0 0 0" xyz="-0.015621881612358529 0.06665620790957599 -0.058074231003688394"/>
+    <mass value="7.368455487741179"/>
+    <inertia ixx="0.018073" ixy="0.000915" ixz="-0.00101" iyy="0.011789" iyz="0.003728" izz="0.01667"/>
+  </inertial>
+  <visual>
+    <origin rpy="0 0 0" xyz="-0.017 -0.3125 -0.115"/>
+    <geometry>
+      <mesh filename="package://spot_arm_description/meshes/Part2_1.stl" scale="0.001 0.001 0.001"/>
+    </geometry>
+    <material name="silver"/>
+  </visual>
+  <collision>
+    <origin rpy="0 0 0" xyz="-0.017 -0.3125 -0.115"/>
+    <geometry>
+      <mesh filename="package://spot_arm_description/meshes/Part2_1.stl" scale="0.001 0.001 0.001"/>
+    </geometry>
+  </collision>
+</link>
+<link name="link4">
   <inertial>
     <origin rpy="0 0 0" xyz="-0.00911464892336129 0.12606054498393937 5.551115123125783e-17"/>
@@ -50,5 +158,25 @@
   </collision>
 </link>
-<link name="gripper_1">
+<link name="wrist">
+  <inertial>
+    <origin rpy="0 0 0" xyz="0.03954999709763633 0.03472006124891969 4.209155544249166e-08"/>
+    <mass value="3.2278801394086396"/>
+    <inertia ixx="0.00339" ixy="-2.1e-05" ixz="0.0" iyy="0.002242" iyz="-0.0" izz="0.003439"/>
+  </inertial>
+  <visual>
+    <origin rpy="0 0 0" xyz="0.0485 -0.69859 -0.0475"/>
+    <geometry>
+      <mesh filename="package://spot_arm_description/meshes/Part4_1.stl" scale="0.001 0.001 0.001"/>
+    </geometry>
+    <material name="silver"/>
+  </visual>
+  <collision>
+    <origin rpy="0 0 0" xyz="0.0485 -0.69859 -0.0475"/>
+    <geometry>
+      <mesh filename="package://spot_arm_description/meshes/Part4_1.stl" scale="0.001 0.001 0.001"/>
+    </geometry>
+  </collision>
+</link>
+<link name="gripper">
   <inertial>
     <origin rpy="0 0 0" xyz="-8.366123908053191e-08 0.07051371901138614 0.017123167388316526"/>
@@ -70,5 +198,5 @@
   </collision>
 </link>
-<link name="finger_1">
+<link name="finger">
   <inertial>
     <origin rpy="0 0 0" xyz="0.8635899028063472 0.09862056591557622 0.00850232975194119"/>
@@ -90,132 +218,3 @@
   </collision>
 </link>
-<link name="Part1_1">
-  <inertial>
-    <origin rpy="0 0 0" xyz="-0.0163095589512068 0.17540914221218962 0.0"/>
-    <mass value="12.658281999999998"/>
-    <inertia ixx="0.12979" ixy="0.002625" ixz="0.0" iyy="0.01004" iyz="0.0" izz="0.129493"/>
-  </inertial>
-  <visual>
-    <origin rpy="0 0 0" xyz="-0.015 -0.0 -0.115"/>
-    <geometry>
-      <mesh filename="package://spot_arm_description/meshes/Part1_1.stl" scale="0.001 0.001 0.001"/>
-    </geometry>
-    <material name="silver"/>
-  </visual>
-  <collision>
-    <origin rpy="0 0 0" xyz="-0.015 -0.0 -0.115"/>
-    <geometry>
-      <mesh filename="package://spot_arm_description/meshes/Part1_1.stl" scale="0.001 0.001 0.001"/>
-    </geometry>
-  </collision>
-</link>
-<link name="Part0_1">
-  <inertial>
-    <origin rpy="0 0 0" xyz="0.05071972800114364 -1.0308563411658574e-17 0.04676911608650795"/>
-    <mass value="6.925827706354272"/>
-    <inertia ixx="0.01241" ixy="-0.0" ixz="-0.001047" iyy="0.010387" iyz="0.0" izz="0.012306"/>
-  </inertial>
-  <visual>
-    <origin rpy="0 0 0" xyz="-0.0 -0.0 -0.065"/>
-    <geometry>
-      <mesh filename="package://spot_arm_description/meshes/Part0_1.stl" scale="0.001 0.001 0.001"/>
-    </geometry>
-    <material name="silver"/>
-  </visual>
-  <collision>
-    <origin rpy="0 0 0" xyz="-0.0 -0.0 -0.065"/>
-    <geometry>
-      <mesh filename="package://spot_arm_description/meshes/Part0_1.stl" scale="0.001 0.001 0.001"/>
-    </geometry>
-  </collision>
-</link>
-<link name="Part4_1">
-  <inertial>
-    <origin rpy="0 0 0" xyz="0.03954999709763633 0.03472006124891969 4.209155544249166e-08"/>
-    <mass value="3.2278801394086396"/>
-    <inertia ixx="0.00339" ixy="-2.1e-05" ixz="0.0" iyy="0.002242" iyz="-0.0" izz="0.003439"/>
-  </inertial>
-  <visual>
-    <origin rpy="0 0 0" xyz="0.0485 -0.69859 -0.0475"/>
-    <geometry>
-      <mesh filename="package://spot_arm_description/meshes/Part4_1.stl" scale="0.001 0.001 0.001"/>
-    </geometry>
-    <material name="silver"/>
-  </visual>
-  <collision>
-    <origin rpy="0 0 0" xyz="0.0485 -0.69859 -0.0475"/>
-    <geometry>
-      <mesh filename="package://spot_arm_description/meshes/Part4_1.stl" scale="0.001 0.001 0.001"/>
-    </geometry>
-  </collision>
-</link>
-<link name="Part2_1">
-  <inertial>
-    <origin rpy="0 0 0" xyz="-0.015621881612358529 0.06665620790957599 -0.058074231003688394"/>
-    <mass value="7.368455487741179"/>
-    <inertia ixx="0.018073" ixy="0.000915" ixz="-0.00101" iyy="0.011789" iyz="0.003728" izz="0.01667"/>
-  </inertial>
-  <visual>
-    <origin rpy="0 0 0" xyz="-0.017 -0.3125 -0.115"/>
-    <geometry>
-      <mesh filename="package://spot_arm_description/meshes/Part2_1.stl" scale="0.001 0.001 0.001"/>
-    </geometry>
-    <material name="silver"/>
-  </visual>
-  <collision>
-    <origin rpy="0 0 0" xyz="-0.017 -0.3125 -0.115"/>
-    <geometry>
-      <mesh filename="package://spot_arm_description/meshes/Part2_1.stl" scale="0.001 0.001 0.001"/>
-    </geometry>
-  </collision>
-</link>
-<joint name="Rev3" type="revolute">
-  <origin rpy="0 0 0" xyz="-0.018 0.138 -0.0675"/>
-  <parent link="Part2_1"/>
-  <child link="Part3_1"/>
-  <axis xyz="0.0 1.0 0.0"/>
-  <limit effort="100" lower="-2.879793" upper="2.879793" velocity="100"/>
-</joint>
-<joint name="Rev6" type="revolute">
-  <origin rpy="0 0 0" xyz="0.04 0.081 0.0"/>
-  <parent link="Part4_1"/>
-  <child link="gripper_1"/>
-  <axis xyz="-0.0 1.0 0.0"/>
-  <limit effort="100" lower="-2.96706" upper="2.96706" velocity="100"/>
-</joint>
-<joint name="Rev7" type="revolute">
-  <origin rpy="0 0 0" xyz="-0.86859 0.043915 -0.029"/>
-  <parent link="gripper_1"/>
-  <child link="finger_1"/>
-  <axis xyz="1.0 -0.0 0.0"/>
-  <limit effort="100" lower="-1.396263" upper="0.349066" velocity="100"/>
-</joint>
-<joint name="Rev8" type="revolute">
-  <origin rpy="0 0 0" xyz="0.015 0.0 0.05"/>
-  <parent link="Part0_1"/>
-  <child link="Part1_1"/>
-  <axis xyz="-1.0 0.0 0.0"/>
-  <limit effort="100" lower="-3.665191" upper="0.0" velocity="100"/>
-</joint>
-<joint name="Rev9" type="revolute">
-  <origin rpy="0 0 0" xyz="0.0 0.0 0.065"/>
-  <parent link="base_link"/>
-  <child link="Part0_1"/>
-  <axis xyz="0.0 0.0 1.0"/>
-  <limit effort="100" lower="-3.141593" upper="2.617994" velocity="100"/>
-</joint>
-<joint name="Rev10" type="revolute">
-  <origin rpy="0 0 0" xyz="-0.0475 0.24809 0.0"/>
-  <parent link="Part3_1"/>
-  <child link="Part4_1"/>
-  <axis xyz="1.0 0.0 0.0"/>
-  <limit effort="100" lower="-1.570796" upper="1.570796" velocity="100"/>
-</joint>
-<joint name="Rev11" type="revolute">
-  <origin rpy="0 0 0" xyz="0.002 0.3125 0.0"/>
-  <parent link="Part1_1"/>
-  <child link="Part2_1"/>
-  <axis xyz="1.0 0.0 0.0"/>
-  <limit effort="100" lower="0.0" upper="2.96706" velocity="100"/>
-</joint>
 </robot>
